Commit message: corrected baxter env

File: gym_baxter_grabbing/envs/cup_urdf.urdf (robot description, URDF)
Before this commit: robot cup, 1 links, 0 joints
Links:
- link base_link: mass 0.00000000001 -> 1; geometry collision mesh filename=mug-9.obj scale=0.005 0.005 0.005; visual mesh filename=mug-9.obj scale=0.005 0.005 0.005

Commit message: modified cup to convex decompo

File: gym_baxter_grabbing/envs/cup_urdf.urdf (robot description, URDF)
Before this commit: robot cup, 1 links, 0 joints
Links:
- link base_link: geometry collision mesh filename=cup.obj scale=0.005 0.005 0.005; visual mesh filename=cup.obj scale=0.005 0.005 0.005
