Commit message: xacro

File: gym_baxter_grabbing/envs/baxter_description/urdf/baxter.urdf.xacro (robot description, xacro)
@@ -4,16 +4,16 @@
   <xacro:arg name="pedestal" default="true"/>
   <!-- Baxter Base URDF -->
-  <xacro:include filename="$(find baxter_description)/urdf/baxter_base/baxter_base.urdf.xacro">
+  <xacro:include filename="baxter_base/baxter_base.urdf.xacro">
     <xacro:arg name="gazebo" value="${gazebo}"/>
   </xacro:include>
   <!-- Baxter Pedestal -->
   <xacro:if value="$(arg pedestal)">
-    <xacro:include filename="$(find baxter_description)/urdf/pedestal/pedestal.xacro">
+    <xacro:include filename="pedestal/pedestal.xacro">
       <xacro:arg name="gazebo" value="${gazebo}"/>
     </xacro:include>
   </xacro:if>
   <!-- Left End Effector -->
-  <xacro:include filename="$(find baxter_description)/urdf/left_end_effector.urdf.xacro" />
+  <xacro:include filename="left_end_effector.urdf.xacro" />
   <!-- Right End Effector -->
-  <xacro:include filename="$(find baxter_description)/urdf/right_end_effector.urdf.xacro" />
+  <xacro:include filename="right_end_effector.urdf.xacro" />
 </robot>

File: gym_baxter_grabbing/envs/baxter_description/urdf/fingers/basic_hard_tip.xacro (robot description, xacro)
@@ -1,4 +1,4 @@
 <?xml version="1.0"?>
-<robot xmlns:xacro="http://www.ros.org/wiki/xacro" name="half_round_tip">
+<robot xmlns:xacro="http://www.ros.org/wiki/xacro" name="basic_hard_tip">
   <xacro:macro name="finger_tip_xacro" params="parent_link reflect grasp *joint_origin">
     <xacro:property name="g_reflect" value="${reflect}" scope="local"/>
@@ -10,5 +10,5 @@
         <origin rpy="0 0 ${pi*(g_reflect+1)/2}" xyz="0 0 0"/>
         <geometry>
-          <mesh filename="package://rethink_ee_description/meshes/electric_gripper/fingers/half_round_tip.DAE" />
+          <mesh filename="package://baxter_description/meshes/electric_gripper/fingers/basic_hard_tip.DAE" />
         </geometry>
       </visual>
@@ -16,5 +16,5 @@
         <origin rpy="0 0 ${pi*(g_reflect+1)/2}" xyz="0 ${-0.0045*g_reflect} -0.015"/>
         <geometry>
-          <cylinder length="0.037" radius="0.008"/>
+          <box size="0.016 0.0065 0.037"/>
         </geometry>
       </collision>

File: gym_baxter_grabbing/envs/baxter_description/urdf/fingers/basic_soft_tip.xacro (robot description, xacro)
@@ -1,4 +1,4 @@
 <?xml version="1.0"?>
-<robot xmlns:xacro="http://www.ros.org/wiki/xacro" name="basic_hard_tip">
+<robot xmlns:xacro="http://www.ros.org/wiki/xacro" name="basic_soft_tip">
   <xacro:macro name="finger_tip_xacro" params="parent_link reflect grasp *joint_origin">
     <xacro:property name="g_reflect" value="${reflect}" scope="local"/>
@@ -10,5 +10,5 @@
         <origin rpy="0 0 ${pi*(g_reflect+1)/2}" xyz="0 0 0"/>
         <geometry>
-          <mesh filename="package://rethink_ee_description/meshes/electric_gripper/fingers/basic_hard_tip.DAE" />
+          <mesh filename="package://baxter_description/meshes/electric_gripper/fingers/basic_soft_tip.DAE" />
         </geometry>
       </visual>
@@ -16,5 +16,5 @@
         <origin rpy="0 0 ${pi*(g_reflect+1)/2}" xyz="0 ${-0.0045*g_reflect} -0.015"/>
         <geometry>
-          <box size="0.016 0.0065 0.037"/>
+          <box size="0.016 0.007 0.037"/>
         </geometry>
       </collision>

File: gym_baxter_grabbing/envs/baxter_description/urdf/fingers/extended_narrow.xacro (robot description, xacro)
@@ -8,5 +8,5 @@
         <origin rpy="0 0 ${-pi/2*(reflect+1)}" xyz="0 0 0"/>
         <geometry>
-          <mesh filename="package://rethink_ee_description/meshes/electric_gripper/fingers/extended_narrow.DAE" />
+          <mesh filename="package://baxter_description/meshes/electric_gripper/fingers/extended_narrow.DAE" />
         </geometry>
       </visual>
@@ -46,5 +46,5 @@
      <xacro:property name="finger_tip" value="none" scope="local"/>
    </xacro:if>
-   <xacro:include filename="$(find rethink_ee_description)/urdf/electric_gripper/fingers/${finger_tip}.xacro" />
+   <xacro:include filename="fingers/${finger_tip}.xacro" />
    <xacro:finger_tip_xacro parent_link="${gripper_side}_gripper_${finger_side}_finger" reflect="${reflect}" grasp="${finger_grasp}">
        <origin rpy="0 0 0" xyz="0.0 ${reflect*finger_width} ${finger_length}"/>

File: gym_baxter_grabbing/envs/baxter_description/urdf/fingers/extended_wide.xacro (robot description, xacro)
@@ -1,18 +1,18 @@
 <?xml version="1.0"?>
-<robot xmlns:xacro="http://www.ros.org/wiki/xacro" name="standard_narrow">
+<robot xmlns:xacro="http://www.ros.org/wiki/xacro" name="wide_extended">
   <xacro:macro name="finger_xacro" params="gripper_side finger_side reflect finger_tip finger_grasp">
-  <xacro:property name="finger_length" value="0.075" scope="global"/>
-  <xacro:property name="finger_width" value="0.01725" scope="local"/>
+    <xacro:property name="finger_length" value="0.1127" scope="global"/>
+    <xacro:property name="finger_width" value="0.05503" scope="local"/>
     <link name="${gripper_side}_gripper_${finger_side}_finger">
       <visual>
         <origin rpy="0 0 ${-pi/2*(reflect+1)}" xyz="0 0 0"/>
         <geometry>
-          <mesh filename="package://rethink_ee_description/meshes/electric_gripper/fingers/standard_narrow.DAE" />
+          <mesh filename="package://baxter_description/meshes/electric_gripper/fingers/extended_wide.DAE" />
         </geometry>
       </visual>
-      <xacro:property name="finger_box_height" value="0.01" scope="local"/>
-      <xacro:property name="finger_box_width" value="0.0135" scope="local"/>
-      <xacro:property name="finger_box_length" value="0.04" scope="local"/>
-      <collision>
+     <xacro:property name="finger_box_height" value="0.01" scope="local"/>
+     <xacro:property name="finger_box_width" value="0.0135" scope="local"/>
+     <xacro:property name="finger_box_length" value="0.0615" scope="local"/>
+     <collision>
         <origin rpy="0 0 ${-pi/2*(reflect+1)}" xyz="0 ${finger_width*reflect} ${finger_box_length}"/>
         <geometry>
@@ -24,5 +24,5 @@
       <xacro:property name="knuckle_box_length" value="${finger_width + 0.03275}" scope="local"/>
       <collision>
-        <origin rpy="0 0 ${-pi/2*(reflect+1)}" xyz="${reflect*-0.005} ${-0.003*reflect} 0.0083"/>
+        <origin rpy="0 0 ${-pi/2*(reflect+1)}" xyz="${reflect*-0.005} ${0.016*reflect} 0.0083"/>
         <geometry>
           <box size="${knuckle_box_height} ${knuckle_box_length} ${knuckle_box_width}"/>
@@ -46,5 +46,5 @@
      <xacro:property name="finger_tip" value="none" scope="local"/>
    </xacro:if>
-   <xacro:include filename="$(find rethink_ee_description)/urdf/electric_gripper/fingers/${finger_tip}.xacro" />
+   <xacro:include filename="fingers/${finger_tip}.xacro" />
    <xacro:finger_tip_xacro parent_link="${gripper_side}_gripper_${finger_side}_finger" reflect="${reflect}" grasp="${finger_grasp}">
        <origin rpy="0 0 0" xyz="0.0 ${reflect*finger_width} ${finger_length}"/>

File: gym_baxter_grabbing/envs/baxter_description/urdf/fingers/half_round_tip.xacro (robot description, xacro)
@@ -1,4 +1,4 @@
 <?xml version="1.0"?>
-<robot xmlns:xacro="http://www.ros.org/wiki/xacro" name="basic_soft_tip">
+<robot xmlns:xacro="http://www.ros.org/wiki/xacro" name="half_round_tip">
   <xacro:macro name="finger_tip_xacro" params="parent_link reflect grasp *joint_origin">
     <xacro:property name="g_reflect" value="${reflect}" scope="local"/>
@@ -10,5 +10,5 @@
         <origin rpy="0 0 ${pi*(g_reflect+1)/2}" xyz="0 0 0"/>
         <geometry>
-          <mesh filename="package://rethink_ee_description/meshes/electric_gripper/fingers/basic_soft_tip.DAE" />
+          <mesh filename="package://baxter_description/meshes/electric_gripper/fingers/half_round_tip.DAE" />
         </geometry>
       </visual>
@@ -16,5 +16,5 @@
         <origin rpy="0 0 ${pi*(g_reflect+1)/2}" xyz="0 ${-0.0045*g_reflect} -0.015"/>
         <geometry>
-          <box size="0.016 0.007 0.037"/>
+          <cylinder length="0.037" radius="0.008"/>
         </geometry>
       </collision>

File: gym_baxter_grabbing/envs/baxter_description/urdf/fingers/paddle_tip.xacro (robot description, xacro)
@@ -10,5 +10,5 @@
         <origin rpy="0 0 ${pi*(g_reflect+1)/2}" xyz="0 0 0"/>
         <geometry>
-          <mesh filename="package://rethink_ee_description/meshes/electric_gripper/fingers/paddle_tip.DAE" />
+          <mesh filename="package://baxter_description/meshes/electric_gripper/fingers/paddle_tip.DAE" />
         </geometry>
       </visual>

File: gym_baxter_grabbing/envs/baxter_description/urdf/fingers/standard_narrow.xacro (robot description, xacro)
@@ -1,18 +1,18 @@
 <?xml version="1.0"?>
-<robot xmlns:xacro="http://www.ros.org/wiki/xacro" name="wide_extended">
+<robot xmlns:xacro="http://www.ros.org/wiki/xacro" name="standard_narrow">
   <xacro:macro name="finger_xacro" params="gripper_side finger_side reflect finger_tip finger_grasp">
-    <xacro:property name="finger_length" value="0.1127" scope="global"/>
-    <xacro:property name="finger_width" value="0.05503" scope="local"/>
+  <xacro:property name="finger_length" value="0.075" scope="global"/>
+  <xacro:property name="finger_width" value="0.01725" scope="local"/>
     <link name="${gripper_side}_gripper_${finger_side}_finger">
       <visual>
         <origin rpy="0 0 ${-pi/2*(reflect+1)}" xyz="0 0 0"/>
         <geometry>
-          <mesh filename="package://rethink_ee_description/meshes/electric_gripper/fingers/extended_wide.DAE" />
+          <mesh filename="package://baxter_description/meshes/electric_gripper/fingers/standard_narrow.DAE" />
         </geometry>
       </visual>
-     <xacro:property name="finger_box_height" value="0.01" scope="local"/>
-     <xacro:property name="finger_box_width" value="0.0135" scope="local"/>
-     <xacro:property name="finger_box_length" value="0.0615" scope="local"/>
-     <collision>
+      <xacro:property name="finger_box_height" value="0.01" scope="local"/>
+      <xacro:property name="finger_box_width" value="0.0135" scope="local"/>
+      <xacro:property name="finger_box_length" value="0.04" scope="local"/>
+      <collision>
         <origin rpy="0 0 ${-pi/2*(reflect+1)}" xyz="0 ${finger_width*reflect} ${finger_box_length}"/>
         <geometry>
@@ -24,5 +24,5 @@
       <xacro:property name="knuckle_box_length" value="${finger_width + 0.03275}" scope="local"/>
       <collision>
-        <origin rpy="0 0 ${-pi/2*(reflect+1)}" xyz="${reflect*-0.005} ${0.016*reflect} 0.0083"/>
+        <origin rpy="0 0 ${-pi/2*(reflect+1)}" xyz="${reflect*-0.005} ${-0.003*reflect} 0.0083"/>
         <geometry>
           <box size="${knuckle_box_height} ${knuckle_box_length} ${knuckle_box_width}"/>
@@ -46,5 +46,5 @@
      <xacro:property name="finger_tip" value="none" scope="local"/>
    </xacro:if>
-   <xacro:include filename="$(find rethink_ee_description)/urdf/electric_gripper/fingers/${finger_tip}.xacro" />
+   <xacro:include filename="fingers/${finger_tip}.xacro" />
    <xacro:finger_tip_xacro parent_link="${gripper_side}_gripper_${finger_side}_finger" reflect="${reflect}" grasp="${finger_grasp}">
        <origin rpy="0 0 0" xyz="0.0 ${reflect*finger_width} ${finger_length}"/>

File: gym_baxter_grabbing/envs/baxter_description/urdf/fingers/standard_wide.xacro (robot description, xacro)
@@ -8,5 +8,5 @@
         <origin rpy="0 0 ${-pi/2*(reflect+1)}" xyz="0 0 0"/>
         <geometry>
-          <mesh filename="package://rethink_ee_description/meshes/electric_gripper/fingers/standard_wide.DAE" />
+          <mesh filename="package://baxter_description/meshes/electric_gripper/fingers/standard_wide.DAE" />
         </geometry>
       </visual>
@@ -46,5 +46,5 @@
      <xacro:property name="finger_tip" value="none" scope="local"/>
    </xacro:if>
-   <xacro:include filename="$(find rethink_ee_description)/urdf/electric_gripper/fingers/${finger_tip}.xacro" />
+   <xacro:include filename="fingers/${finger_tip}.xacro" />
    <xacro:finger_tip_xacro parent_link="${gripper_side}_gripper_${finger_side}_finger" reflect="${reflect}" grasp="${finger_grasp}">
        <origin rpy="0 0 0" xyz="0.0 ${reflect*finger_width} ${finger_length}"/>

File: gym_baxter_grabbing/envs/baxter_description/urdf/generated/extended_narrow_3_paddle_inner.urdf (robot description, URDF)
Before this commit: robot baxter, 44 links, 43 joints
Links:
- added link l_gripper_l_finger, mass 0.02; collision box size=0.01 0.0135 0.1127; collision box size=0.01 0.05 0.017
- added link l_gripper_l_finger_tip, mass 0.01; collision box size=0.042 0.0065 0.037; visual mesh filename=package://baxter_description/meshes/electric_gripper/finger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
- added link l_gripper_r_finger, mass 0.02; collision box size=0.01 0.0135 0.1127; collision box size=0.01 0.05 0.017
- added link l_gripper_r_finger_tip, mass 0.01; collision box size=0.042 0.0065 0.037; visual mesh filename=package://baxter_description/meshes/electric_gripper/finger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
- added link left_gripper, mass 0.0001
- added link left_gripper_base, mass 0.3; collision cylinder length=0.1 radius=0.029; visual mesh filename=package://baxter_description/meshes/electric_gripper/electr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
- added link pedestal, mass 60.86397744; collision mesh filename=package://baxter_description/meshes/base/pedestal_link_coll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; visual mesh filename=package://baxter_description/meshes/base/PEDESTAL.DAE
- added link r_gripper_l_finger, mass 0.02; collision box size=0.01 0.0135 0.1127; collision box size=0.01 0.05 0.017
- added link r_gripper_l_finger_tip, mass 0.01; collision box size=0.042 0.0065 0.037; visual mesh filename=package://baxter_description/meshes/electric_gripper/finger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
- added link r_gripper_r_finger, mass 0.02; collision box size=0.01 0.0135 0.1127; collision box size=0.01 0.05 0.017
- added link r_gripper_r_finger_tip, mass 0.01; collision box size=0.042 0.0065 0.037; visual mesh filename=package://baxter_description/meshes/electric_gripper/finger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
- added link right_gripper, mass 0.0001
- added link right_gripper_base, mass 0.3; collision cylinder length=0.1 radius=0.029; visual mesh filename=package://baxter_description/meshes/electric_gripper/electr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
Joints:
- added joint l_gripper_l_finger_joint: type prismatic, parent left_gripper_base, child l_gripper_l_finger, origin xyz=0.0 0.008 0.02 rpy=0 0 0, axis 0 1 0, limit lower=0.0 upper=0.020833 effort=20.0 velocity=5.0
- added joint l_gripper_l_finger_tip_joint: type fixed, parent l_gripper_l_finger, child l_gripper_l_finger_tip, origin xyz=0.0 0.01725 0.1127 rpy=0 0 0
- added joint l_gripper_r_finger_joint: type prismatic, parent left_gripper_base, child l_gripper_r_finger, origin xyz=0.0 -0.008 0.02 rpy=0 0 0, axis 0 1 0, limit lower=-0.020833 upper=0.0 effort=20.0 velocity=5.0, mimic joint=l_gripper_l_finger_joint multiplier=-1.0
- added joint l_gripper_r_finger_tip_joint: type fixed, parent l_gripper_r_finger, child l_gripper_r_finger_tip, origin xyz=0.0 -0.01725 0.1127 rpy=0 0 0
- added joint left_endpoint: type fixed, parent left_gripper_base, child left_gripper, origin xyz=0 0 0.13269999999999998 rpy=0 0 0
- added joint left_gripper_base: type fixed, parent left_hand, child left_gripper_base, origin xyz=0 0 0.025 rpy=0 0 0
- added joint pedestal_fixed: type fixed, parent torso, child pedestal, origin xyz=0.0 0.0 0.0 rpy=0 0 0
- added joint r_gripper_l_finger_joint: type prismatic, parent right_gripper_base, child r_gripper_l_finger, origin xyz=0.0 0.008 0.02 rpy=0 0 0, axis 0 1 0, limit lower=0.0 upper=0.020833 effort=20.0 velocity=5.0
- added joint r_gripper_l_finger_tip_joint: type fixed, parent r_gripper_l_finger, child r_gripper_l_finger_tip, origin xyz=0.0 0.01725 0.1127 rpy=0 0 0
- added joint r_gripper_r_finger_joint: type prismatic, parent right_gripper_base, child r_gripper_r_finger, origin xyz=0.0 -0.008 0.02 rpy=0 0 0, axis 0 1 0, limit lower=-0.020833 upper=0.0 effort=20.0 velocity=5.0, mimic joint=r_gripper_l_finger_joint multiplier=-1.0
- added joint r_gripper_r_finger_tip_joint: type fixed, parent r_gripper_r_finger, child r_gripper_r_finger_tip, origin xyz=0.0 -0.01725 0.1127 rpy=0 0 0
- added joint right_endpoint: type fixed, parent right_gripper_base, child right_gripper, origin xyz=0 0 0.13269999999999998 rpy=0 0 0
- added joint right_gripper_base: type fixed, parent right_hand, child right_gripper_base, origin xyz=0 0 0.025 rpy=0 0 0

File: gym_baxter_grabbing/envs/baxter_description/urdf/left_end_effector.urdf.xacro (robot description, xacro)
@@ -1,13 +1,13 @@
 <?xml version="1.0" ?>
-<robot name="right_end_effector" xmlns:xacro="http://www.ros.org/wiki/xacro">
-  <xacro:include filename="$(find rethink_ee_description)/urdf/electric_gripper/rethink_electric_gripper.xacro" />
-  <xacro:rethink_electric_gripper side="right"
+<robot name="left_end_effector" xmlns:xacro="http://www.ros.org/wiki/xacro">
+  <xacro:include filename="rethink_electric_gripper.xacro" />
+  <xacro:rethink_electric_gripper side="left"
                                   l_finger="extended_narrow"
                                   l_finger_slot="2"
-                                  l_finger_tip="half_round_tip"
+                                  l_finger_tip="paddle_tip"
                                   l_finger_grasp="inner"
                                   r_finger="extended_narrow"
                                   r_finger_slot="2"
-                                  r_finger_tip="half_round_tip"
+                                  r_finger_tip="paddle_tip"
                                   r_finger_grasp="inner"/>
 </robot>

File: gym_baxter_grabbing/envs/baxter_description/urdf/pedestal/pedestal.xacro (robot description, xacro)
@@ -1,4 +1,4 @@
 <?xml version="1.0" ?>
-<robot name="pedistal" xmlns:xacro="http://www.ros.org/wiki/xacro">
+<robot name="pedestal" xmlns:xacro="http://www.ros.org/wiki/xacro">
   <!-- Arguments and Defaults-->
   <xacro:arg name="gazebo" default="false"/>

File: gym_baxter_grabbing/envs/baxter_description/urdf/rethink_electric_gripper.xacro (robot description, xacro)
@@ -8,5 +8,5 @@
         <origin rpy="${-pi/2} ${pi} 0" xyz="0 0 0"/>
         <geometry>
-          <mesh filename="package://rethink_ee_description/meshes/electric_gripper/electric_gripper_base.DAE"/>
+          <mesh filename="package://baxter_description/meshes/electric_gripper/electric_gripper_base.DAE"/>
         </geometry>
       </visual>
@@ -28,9 +28,9 @@
     <!-- Left finger link -->
     <xacro:property name="finger_length" value="0.0" scope="global"/>
-    <xacro:include filename="$(find rethink_ee_description)/urdf/electric_gripper/fingers/${l_finger}.xacro" />
+    <xacro:include filename="fingers/${l_finger}.xacro" />
     <xacro:finger_xacro gripper_side="${gripper_side}" finger_side="l" reflect="1" finger_tip="${l_finger_tip}" finger_grasp="${l_finger_grasp}"/>
     <xacro:property name="tip_finger_length" value="${finger_length}" scope="local"/>
     <!-- Right finger link -->
-    <xacro:include filename="$(find rethink_ee_description)/urdf/electric_gripper/fingers/${r_finger}.xacro" />
+    <xacro:include filename="fingers/${r_finger}.xacro" />
     <xacro:finger_xacro gripper_side="${gripper_side}" finger_side="r" reflect="-1" finger_tip="${r_finger_tip}" finger_grasp="${r_finger_grasp}"/>
     <xacro:if value="${finger_length > tip_finger_length}">

File: gym_baxter_grabbing/envs/baxter_description/urdf/right_end_effector.urdf.xacro (robot description, xacro)
@@ -1,13 +1,13 @@
 <?xml version="1.0" ?>
-<robot name="left_end_effector" xmlns:xacro="http://www.ros.org/wiki/xacro">
-  <xacro:include filename="$(find rethink_ee_description)/urdf/electric_gripper/rethink_electric_gripper.xacro" />
-  <xacro:rethink_electric_gripper side="left"
+<robot name="right_end_effector" xmlns:xacro="http://www.ros.org/wiki/xacro">
+  <xacro:include filename="rethink_ee_description/urdf/electric_gripper/rethink_electric_gripper.xacro" />
+  <xacro:rethink_electric_gripper side="right"
                                   l_finger="extended_narrow"
                                   l_finger_slot="2"
-                                  l_finger_tip="paddle_tip"
+                                  l_finger_tip="half_round_tip"
                                   l_finger_grasp="inner"
                                   r_finger="extended_narrow"
                                   r_finger_slot="2"
-                                  r_finger_tip="paddle_tip"
+                                  r_finger_tip="half_round_tip"
                                   r_finger_grasp="inner"/>
 </robot>
