Commit message: s1

File: gym_baxter_grabbing/envs/robots/baxter_description/urdf/baxter_base/baxter_base.urdf.xacro (robot description, xacro)
@@ -532,5 +532,5 @@
     <parent link="right_upper_shoulder"/>
     <child link="right_lower_shoulder"/>
-    <limit effort="${max(50.0*$(arg limit_scale),50.0)}" lower="-2.147" upper="1.047" velocity="${1.5*$(arg limit_scale)}"/>
+    <limit effort="${max(50.0*$(arg limit_scale),100.0)}" lower="-2.147" upper="1.047" velocity="${1.5*$(arg limit_scale)}"/>
     <dynamics damping="0.7" friction="0.0"/>
   </joint>
@@ -900,5 +900,5 @@
     <parent link="left_upper_shoulder"/>
     <child link="left_lower_shoulder"/>
-    <limit effort="${max(50.0*$(arg limit_scale),50.0)}" lower="-2.147" upper="1.047" velocity="${1.5*$(arg limit_scale)}"/>
+    <limit effort="${max(50.0*$(arg limit_scale),100.0)}" lower="-2.147" upper="1.047" velocity="${1.5*$(arg limit_scale)}"/>
     <dynamics damping="0.7" friction="0.0"/>
   </joint>
